File: dorne/pcb/dorne.kicad_pcb (KiCad board)
At the start: 2 copper layers, 275.5 x 105.6 mm, 172 parts, among them J1 MJ-4PP-9, J2 OLED, J3 MJ-4PP-9, J4 OLED, SW1 SW_PUSH, SW10 SW_PUSH, SW11 SW_PUSH, SW12 SW_PUSH, SW13 SW_PUSH, SW14 SW_PUSH, SW15 SW_PUSH, SW16 SW_PUSH, SW17 SW_PUSH, SW18 SW_PUSH, SW19 SW_PUSH, SW2 SW_PUSH, SW20 SW_PUSH, SW21 SW_PUSH, SW22 SW_PUSH, SW23 SW_PUSH, SW24 SW_PUSH, SW25 SW_PUSH, SW26 SW_PUSH, SW27 SW_PUSH, SW28 SW_PUSH, SW29 SW_PUSH, SW3 SW_PUSH, SW30 SW_PUSH, SW31 SW_PUSH, SW32 SW_PUSH, SW33 SW_PUSH, SW34 SW_PUSH, SW35 SW_PUSH, SW36 SW_PUSH, SW37 SW_PUSH, SW38 SW_PUSH, SW39 SW_PUSH, SW4 SW_PUSH, SW40 SW_PUSH, SW41 SW_PUSH, SW42 SW_PUSH, SW5 SW_PUSH, SW6 SW_PUSH, SW7 SW_PUSH, SW8 SW_PUSH, SW9 SW_PUSH, U1 ProMicro, U2 ProMicro

Commit message: RM LEDs
Parts:
- removed G*** (x4): LOGO, kbd:corne-logo-horizontal
- removed LED1, LED2, LED28, LED29, LED3, LED30, LED31, LED32, LED33, LED4, LED5, LED6: WS2812B, LED_SMD:LED_WS2812B_PLCC4_5.0x5.0mm_P3.2mm
- removed LED10, LED11, LED12, LED13, LED14, LED15, LED16, LED17, LED18, LED19, LED20, LED21, LED22, LED23, LED24, LED25, LED26, LED27, LED34, LED35, LED36, LED37, LED38, LED39, LED40, LED41, LED42, LED43, LED44, LED45, LED46, LED47, LED48, LED49, LED50, LED51, LED52, LED53, LED54, LED7, LED8, LED9: YS-SK6812MINI-E, kbd:YS-SK6812MINI-E
- removed REF** (x8): Breakaway_Tabs, kbd:Breakaway_Tabs
- removed Ref** (x14): Val**, kbd:M2_HOLE_v2
Connections:
- J1 pad A: Net-(J1-PadA) -> unconnected-(J1-PadA)
- J3 pad A: Net-(J3-PadA) -> unconnected-(J3-PadA)
- U1 pad 11: Net-(U1-Pad11) -> unconnected-(U1-Pad11)
- U1 pad 12: Net-(U1-Pad12) -> unconnected-(U1-Pad12)
- U1 pad 13: Net-(U1-Pad13) -> unconnected-(U1-Pad13)
- U1 pad 14: Net-(U1-Pad14) -> unconnected-(U1-Pad14)
- U1 pad 24: Net-(U1-Pad24) -> unconnected-(U1-Pad24)
- U2 pad 11: Net-(U2-Pad11) -> unconnected-(U2-Pad11)
- U2 pad 12: Net-(U2-Pad12) -> unconnected-(U2-Pad12)
- U2 pad 13: Net-(U2-Pad13) -> unconnected-(U2-Pad13)
- U2 pad 14: Net-(U2-Pad14) -> unconnected-(U2-Pad14)
- U2 pad 24: Net-(U2-Pad24) -> unconnected-(U2-Pad24)
Routing:
- net GND: track 637.2 -> 66.1 mm, vias 16 -> 0
- net GNDA: track 617.9 -> 77.7 mm, vias 15 -> 0
- net VDD: track 573.1 -> 41.2 mm, vias 2 -> 0
- net VCC: track 544.3 -> 48.8 mm, vias 2 -> 0
- net Net-(LED31-Pad2): track 71.8 -> 0.00 mm, vias 2 -> 0
- net Net-(LED1-Pad4): track 47.8 -> 0.00 mm
- net Net-(LED32-Pad2): track 47.4 -> 0.00 mm
- net Net-(LED2-Pad4): track 46.3 -> 0.00 mm
- net Net-(LED4-Pad2): track 43.6 -> 0.00 mm, vias 2 -> 0
- net Net-(LED28-Pad2): track 41.5 -> 0.00 mm, vias 2 -> 0
- net LED: track 41.1 -> 0.00 mm
- net Net-(LED20-Pad4): track 36.8 -> 0.00 mm, vias 4 -> 0
- net Net-(LED29-Pad4): track 36.4 -> 0.00 mm
- net Net-(LED24-Pad4): track 36.0 -> 0.00 mm, vias 2 -> 0
- net Net-(LED28-Pad4): track 35.9 -> 0.00 mm
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