File: dorne/pcb/dorne.kicad_pcb (KiCad board)
At the start: 2 copper layers, 275.5 x 105.6 mm, 92 parts, among them J1 MJ-4PP-9, J2 OLED, J3 MJ-4PP-9, J4 OLED, SW1 SW_PUSH, SW10 SW_PUSH, SW11 SW_PUSH, SW12 SW_PUSH, SW13 SW_PUSH, SW14 SW_PUSH, SW15 SW_PUSH, SW16 SW_PUSH, SW17 SW_PUSH, SW18 SW_PUSH, SW19 SW_PUSH, SW2 SW_PUSH, SW20 SW_PUSH, SW21 SW_PUSH, SW22 SW_PUSH, SW23 SW_PUSH, SW24 SW_PUSH, SW25 SW_PUSH, SW26 SW_PUSH, SW27 SW_PUSH, SW28 SW_PUSH, SW29 SW_PUSH, SW3 SW_PUSH, SW30 SW_PUSH, SW31 SW_PUSH, SW32 SW_PUSH, SW33 SW_PUSH, SW34 SW_PUSH, SW35 SW_PUSH, SW36 SW_PUSH, SW37 SW_PUSH, SW38 SW_PUSH, SW39 SW_PUSH, SW4 SW_PUSH, SW40 SW_PUSH, SW41 SW_PUSH, SW42 SW_PUSH, SW5 SW_PUSH, SW6 SW_PUSH, SW7 SW_PUSH, SW8 SW_PUSH, SW9 SW_PUSH, U1 ProMicro, U2 ProMicro

Commit message: cherry->choc
Parts:
- SW1, SW10, SW11, SW12, SW13, SW14, SW15, SW16, SW17, SW18, SW19, SW2, SW20, SW22, SW23, SW24, SW25, SW26, SW27, SW28, SW29, SW3, SW30, SW31, SW32, SW33, SW34, SW35, SW36, SW37, SW38, SW39, SW4, SW40, SW41, SW5, SW6, SW7, SW8, SW9: footprint kbd:CherryMX_Hotswap -> kbd:ChocV1_V2_Hotswap
- SW21, SW42: footprint kbd:CherryMX_Hotswap_1.5u -> kbd:ChocV1_V2_Hotswap_1.5u
- moved D19 39.1 mm to (115.1, 92.1), turned to -90 degrees
- moved D21 38.4 mm to (136.4, 87.0), turned to 0 degrees
- moved D42 23.9 mm to (172.9, 89.8), turned to -90 degrees
- moved D41 2.46 mm to (197.2, 89.0), turned to -90 degrees
- moved D22 0.13 mm to (284.2, 35.9), turned to -90 degrees
- turned D1 to -90 degrees
- turned D10 to -90 degrees
- turned D11 to -90 degrees
- turned D12 to -90 degrees
- turned D13 to -90 degrees
- turned D14 to -90 degrees
- turned D15 to -90 degrees
- turned D16 to -90 degrees
- turned D17 to -90 degrees
- turned D18 to -90 degrees
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Connections:
- D19 pad 2: Net-(D19-Pad2) -> Net-(D20-Pad2)
- D20 pad 2: Net-(D20-Pad2) -> Net-(D19-Pad2)
Routing:
- net row2: track 180.3 -> 135.2 mm, vias 2 -> 0
- net row0: track 182.7 -> 138.7 mm, vias 2 -> 0
- net row0_r: track 184.4 -> 143.4 mm
- net row1_r: track 166.2 -> 125.3 mm
- net row2_r: track 172.0 -> 134.0 mm
- net row1: track 193.1 -> 155.4 mm
- net row3: track 121.6 -> 89.5 mm
- net Net-(D21-Pad2): track 38.3 -> 8.93 mm
- net Net-(D42-Pad2): track 33.7 -> 15.0 mm
- net col0_r: track 175.8 -> 157.4 mm, vias 5 -> 4
- net Net-(D20-Pad2): track 23.7 -> 7.55 mm
- net Net-(D19-Pad2): track 22.2 -> 6.92 mm
- net row3_r: track 95.3 -> 81.7 mm
- net col1_r: track 150.6 -> 137.9 mm
- net col1: track 149.3 -> 138.2 mm
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