File: dorne/pcb/dorne.kicad_pcb (KiCad board)
At the start: 2 copper layers, 275.5 x 105.6 mm, 102 parts, among them J1 MJ-4PP-9, J2 MJ-4PP-9, SW1 SW_PUSH, SW10 SW_PUSH, SW11 SW_PUSH, SW12 SW_PUSH, SW13 SW_PUSH, SW14 SW_PUSH, SW15 SW_PUSH, SW16 SW_PUSH, SW17 SW_PUSH, SW18 SW_PUSH, SW19 SW_PUSH, SW2 SW_PUSH, SW20 SW_PUSH, SW21 SW_PUSH, SW22 SW_PUSH, SW23 SW_PUSH, SW24 SW_PUSH, SW25 SW_PUSH, SW26 SW_PUSH, SW27 SW_PUSH, SW28 SW_PUSH, SW29 SW_PUSH, SW3 SW_PUSH, SW30 SW_PUSH, SW31 SW_PUSH, SW32 SW_PUSH, SW33 SW_PUSH, SW34 SW_PUSH, SW35 SW_PUSH, SW36 SW_PUSH, SW37 SW_PUSH, SW38 SW_PUSH, SW39 SW_PUSH, SW4 SW_PUSH, SW40 SW_PUSH, SW41 SW_PUSH, SW42 SW_PUSH, SW5 SW_PUSH, SW6 SW_PUSH, SW7 SW_PUSH, SW8 SW_PUSH, SW9 SW_PUSH, U3 nice_nano, U4 nice_nano

Commit message: Realigned everything!!!!
Parts:
- added Ref**: Val**, kbd:M2_HOLE_v2, F.Cu at (167.4, 45.0)
- added Ref**: Val**, kbd:M2_HOLE_v2, F.Cu at (89.3, 57.4)
- added Ref**: Val**, kbd:M2_HOLE_v2, F.Cu at (91.4, 48.5)
- added Ref**: Val**, kbd:M2_HOLE_v2, B.Cu at (217.7, 86.0)
- added Ref**: Val**, kbd:M2_HOLE_v2, B.Cu at (332.4, 57.4)
- added Ref**: Val**, kbd:M2_HOLE_v2, B.Cu at (232.1, 77.5)
- added Ref**: Val**, kbd:M2_HOLE_v2, F.Cu at (134.6, 84.7)
- added Ref**: Val**, kbd:M2_HOLE_v2, F.Cu at (181.1, 92.4)
- added Ref**: Val**, kbd:M2_HOLE_v2, F.Cu at (189.7, 77.5)
- added Ref**: Val**, kbd:M2_HOLE_v2, F.Cu at (204.1, 86.0)
- added Ref**: Val**, kbd:M2_HOLE_v2, F.Cu at (240.6, 92.4)
- added Ref**: Val**, kbd:M2_HOLE_v2, F.Cu at (287.2, 84.8)
- added Ref**: Val**, kbd:M2_HOLE_v2, F.Cu at (330.3, 48.5)
- added Ref**: Val**, kbd:M2_HOLE_v2, F.Cu at (254.4, 45.0)
- moved H3 63.5 mm to (228.0, 40.0)
- moved D41 63.3 mm to (260.5, 91.7)
- moved G*** 63.3 mm to (301.9, 85.0) (x2)
- moved SW24 63.3 mm to (301.9, 34.2)
- moved SW25 63.3 mm to (282.9, 31.9)
- moved SW26 63.3 mm to (263.9, 34.2)
- moved SW30 63.3 mm to (301.9, 53.2)
- moved SW31 63.3 mm to (282.9, 50.9)
- moved SW32 63.3 mm to (263.9, 53.2)
- moved SW36 63.3 mm to (301.9, 72.2)
- moved SW37 63.3 mm to (282.9, 69.9)
- moved SW38 63.3 mm to (263.9, 72.2)
- moved SW40 63.3 mm to (273.4, 91.9)
- moved D22 63.3 mm to (347.5, 39.1)
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Routing:
- net row3: track 96.0 -> 101.6 mm
- net Net-(D20-Pad2): track 12.7 -> 7.64 mm
- net col1: track 165.8 -> 168.1 mm
- net data_r: track 63.5 -> 65.1 mm
- net row1_r: track 151.0 -> 149.4 mm
- net bat_pos_r: track 40.3 -> 41.8 mm
- net col5: track 102.0 -> 103.5 mm
- net col4_r: track 112.2 -> 113.6 mm
- net row2_r: track 159.5 -> 158.3 mm
- net GNDA: track 75.4 -> 76.4 mm
- net GND: track 62.5 -> 63.4 mm
- net col0_r: track 179.9 -> 179.1 mm
- net data: track 76.8 -> 77.5 mm
- net reset_r: track 26.7 -> 27.3 mm
- net VCC: track 45.2 -> 45.7 mm
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Other:
- board size 275.5 x 105.6 mm -> 277.8 x 91.4 mm
