File: dorne/pcb/dorne.kicad_pcb (KiCad board)
At the start: 2 copper layers, 277.8 x 91.4 mm, 116 parts, among them J1 MJ-4PP-9, J2 MJ-4PP-9, SW1 SW_PUSH, SW10 SW_PUSH, SW11 SW_PUSH, SW12 SW_PUSH, SW13 SW_PUSH, SW14 SW_PUSH, SW15 SW_PUSH, SW16 SW_PUSH, SW17 SW_PUSH, SW18 SW_PUSH, SW19 SW_PUSH, SW2 SW_PUSH, SW20 SW_PUSH, SW21 SW_PUSH, SW22 SW_PUSH, SW23 SW_PUSH, SW24 SW_PUSH, SW25 SW_PUSH, SW26 SW_PUSH, SW27 SW_PUSH, SW28 SW_PUSH, SW29 SW_PUSH, SW3 SW_PUSH, SW30 SW_PUSH, SW31 SW_PUSH, SW32 SW_PUSH, SW33 SW_PUSH, SW34 SW_PUSH, SW35 SW_PUSH, SW36 SW_PUSH, SW37 SW_PUSH, SW38 SW_PUSH, SW39 SW_PUSH, SW4 SW_PUSH, SW40 SW_PUSH, SW41 SW_PUSH, SW42 SW_PUSH, SW5 SW_PUSH, SW6 SW_PUSH, SW7 SW_PUSH, SW8 SW_PUSH, SW9 SW_PUSH, U3 nice_nano, U4 nice_nano

Commit message: I think it's done?
Parts:
- removed the Ref** at (89.3, 57.4)
- removed the Ref** at (217.7, 86.0)
- removed the Ref** at (332.4, 57.4)
- removed the Ref** at (232.1, 77.5)
- removed the Ref** at (189.7, 77.5)
- removed the Ref** at (204.1, 86.0)
- added Ref**: Val**, kbd:M2_HOLE_v2, F.Cu at (91.4, 67.5)
- added Ref**: Val**, kbd:M2_HOLE_v2, F.Cu at (231.5, 77.0)
- added Ref**: Val**, kbd:M2_HOLE_v2, F.Cu at (330.4, 67.5)
- added Ref**: Val**, kbd:M2_HOLE_v2, F.Cu at (190.2, 77.0)
- moved Ref** 0.39 mm to (240.8, 92.0)
- moved Ref** 0.38 mm to (181.0, 92.0)
- moved Ref** 0.06 mm to (287.2, 84.8)
- moved Ref** 0.06 mm to (134.5, 84.8)
Routing:
- net row3_r: track 86.2 -> 86.9 mm

Commit message: JLC Submitted versino
Parts:
- added REF**: Breakaway_Tabs, kbd:Breakaway_Tabs, F.Cu at (206.9, 37.5)
- added REF**: Breakaway_Tabs, kbd:Breakaway_Tabs, F.Cu at (206.9, 61.5)
- added REF**: Breakaway_Tabs, kbd:Breakaway_Tabs, F.Cu at (214.9, 83.5)
- added REF**: Breakaway_Tabs, kbd:Breakaway_Tabs, F.Cu at (206.9, 83.5)
- added REF**: Breakaway_Tabs, kbd:Breakaway_Tabs, F.Cu at (214.9, 37.5)
- added REF**: Breakaway_Tabs, kbd:Breakaway_Tabs, F.Cu at (214.9, 61.5)
- moved PSW0 0.15 mm to (196.9, 32.0)
- moved PSW1 0.10 mm to (225.1, 32.0)
Other:
- outline, holes or cut-outs redrawn

Commit message: Saving so I can look at my old files
Parts:
- removed D22, D23, D24, D25, D26, D27, D28, D29, D30, D31, D32, D33, D34, D35, D36, D37, D38, D39, D40, D41, D42: D, kbd:D3_SMD_v2
- removed G*** (x2): LOGO, lib:dorne-logo-horizontal
- removed H2, H3: MountingHole_Pad, Connector_Pin:Pin_D1.0mm_L10.0mm
- removed J2: MJ-4PP-9, kbd:MJ-4PP-9_1side
- removed PSW1: SW_SPDT, lib:ALPS-SSSS811101-0
- removed PSW3: SW_SPST, buttons:SW_L068-A
- removed REF** (x6): Breakaway_Tabs, kbd:Breakaway_Tabs
- removed RSW2: SW_PUSH, lib:CK_Components-KSR223GNCLFG-0
- removed Ref** (x6): Val**, kbd:M2_HOLE_v2
- removed SW22, SW23, SW24, SW25, SW26, SW27, SW28, SW29, SW30, SW31, SW32, SW33, SW34, SW35, SW36, SW37, SW38, SW39, SW40, SW41: SW_PUSH, kbd:ChocV1_V2_Hotswap
- removed SW42: SW_PUSH, kbd:ChocV1_V2_Hotswap_1.5u
- removed U4: nice_nano, nicenano:nice_nano
- moved D1 1.39 mm to (90.5, 38.0)
- renumbered G*** to LOGO1, G*** to LOGO2, Ref** to MH1, Ref** to MH2, Ref** to MH3, Ref** to MH4, Ref** to MH5, Ref** to MH6
Routing:
- net col0_r: track 179.3 -> 0.00 mm, vias 6 -> 0
- net row0_r: track 170.5 -> 0.00 mm, vias 1 -> 0
- net col1_r: track 164.0 -> 0.00 mm, vias 6 -> 0
- net row2_r: track 158.4 -> 0.00 mm
- net row1_r: track 149.4 -> 0.00 mm
- net col3_r: track 124.9 -> 0.00 mm, vias 7 -> 0
- net col2_r: track 118.4 -> 0.00 mm, vias 5 -> 0
- net col4_r: track 113.6 -> 0.00 mm, vias 7 -> 0
- net row3_r: track 86.9 -> 0.00 mm
- net col5_r: track 85.1 -> 0.00 mm, vias 7 -> 0
- net GNDA: track 76.6 -> 0.00 mm
- net data_r: track 65.3 -> 0.00 mm
- net VDD: track 47.6 -> 0.00 mm, vias 2 -> 0
- net bat_pos_r: track 41.8 -> 0.00 mm
- net bat_in_r: track 40.9 -> 0.00 mm, vias 1 -> 0
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Other:
- board size 277.8 x 91.4 mm -> 134.8 x 91.4 mm
